Commit message: mocked robot_arm and robot_base works

File: peerajak_ros2_control_robot_description/urdf/mobile_base.ros2_control.xacro (robot description, xacro)
@@ -1,12 +1,12 @@
 <?xml version="1.0"?>
 <robot xmlns:xacro="http://www.ros.org/wiki/xacro">
-    <ros2_control name="MobileBase" type="system">
+    <ros2_control name="MobileBaseOnly" type="system">
         <hardware>
-            <!-- <plugin>mock_components/GenericSystem</plugin>
-            <param name="calculate_dynamics">true</param> -->
-            <plugin>mobile_base_hardware/MobileBaseHardwareInterface</plugin>
+            <plugin>mock_components/GenericSystem</plugin>
+            <param name="calculate_dynamics">true</param>
+            <!-- plugin>mobile_base_hardware/MobileBaseHardwareInterface</plugin>
             <param name="left_motor_id">10</param>
             <param name="right_motor_id">20</param>
-            <param name="dynamixel_port">/dev/ttyACM0</param>
+            <param name="dynamixel_port">/dev/ttyACM0</param -->
         </hardware>
         <joint name="base_right_wheel_joint">

File: peerajak_ros2_control_robot_description/urdf/mobile_base.xacro (robot description, xacro)
@@ -1,6 +1,6 @@
 <?xml version="1.0"?>
 <robot xmlns:xacro="http://www.ros.org/wiki/xacro">
-  <!-- Include ros2_control Plugins -->
-  <xacro:include filename="$(find peerajak_ros2_control_robot_description)/urdf/mobile_base.ros2_control.xacro" />
+  <!-- Include ros2_control Plugins
+  <xacro:include filename="$(find peerajak_ros2_control_robot_description)/urdf/mobile_base.ros2_control.xacro" /> -->
     <xacro:property name="base_length" value="0.6" />
     <xacro:property name="base_width" value="0.4" />

File: peerajak_ros2_control_robot_description/urdf/peerajak_ros2_control_robot.urdf.xacro (robot description, xacro)
@@ -1,5 +1,13 @@
 <?xml version="1.0"?>
-<robot name="peerajak_ros2_control_robot" xmlns:xacro="http://www.ros.org/wiki/xacro">
+<robot name="my_robot" xmlns:xacro="http://www.ros.org/wiki/xacro">
     <xacro:include filename="common_properties.xacro" />
     <xacro:include filename="mobile_base.xacro" />
+    <xacro:include filename="mobile_base.ros2_control.xacro" />
+    <xacro:include filename="arm.xacro"/>
+    <xacro:include filename="arm.ros2_control.xacro"/>
+    <joint name="mobile_base_arm_joint" type="fixed">
+        <parent link="base_link" />
+        <child link="arm_base_link" />
+        <origin xyz="${base_length / 4.0} 0 ${base_height}" rpy="0 0 0" />
+    </joint>
 </robot>
